File: core_holder/core_holder.kicad_pcb (KiCad board)
At the start: 2 copper layers, 149.4 x 149.4 mm, 8 parts

Commit message: finalising
Parts:
- added REF**: Pin_Header_Straight_1x01_Pitch2.54mm, Pin_Headers:Pin_Header_Straight_1x01_Pitch2.54mm, F.Cu at (148.6, 55.8)
- added REF**: Pin_Header_Straight_1x01_Pitch2.54mm, Pin_Headers:Pin_Header_Straight_1x01_Pitch2.54mm, F.Cu at (148.6, 111.2)
- added REF** (x2): Pin_Header_Straight_1x01_Pitch2.54mm, Pin_Headers:Pin_Header_Straight_1x01_Pitch2.54mm, F.Cu at (178.3, 76.2)
- added REF**: Pin_Header_Straight_1x01_Pitch2.54mm, Pin_Headers:Pin_Header_Straight_1x01_Pitch2.54mm, F.Cu at (179.5, 81.2)
- added REF**: Pin_Header_Straight_1x01_Pitch2.54mm, Pin_Headers:Pin_Header_Straight_1x01_Pitch2.54mm, F.Cu at (180.2, 86.3)
- added REF**: Pin_Header_Straight_1x01_Pitch2.54mm, Pin_Headers:Pin_Header_Straight_1x01_Pitch2.54mm, F.Cu at (180.6, 91.2)
- added REF**: Pin_Header_Straight_1x01_Pitch2.54mm, Pin_Headers:Pin_Header_Straight_1x01_Pitch2.54mm, F.Cu at (180.7, 96.3)
- added REF**: Pin_Header_Straight_1x01_Pitch2.54mm, Pin_Headers:Pin_Header_Straight_1x01_Pitch2.54mm, F.Cu at (180.3, 101.3)
- added REF**: Pin_Header_Straight_1x01_Pitch2.54mm, Pin_Headers:Pin_Header_Straight_1x01_Pitch2.54mm, F.Cu at (179.6, 106.2)
- added REF**: Pin_Header_Straight_1x01_Pitch2.54mm, Pin_Headers:Pin_Header_Straight_1x01_Pitch2.54mm, F.Cu at (178.6, 111.2)
- added REF**: Pin_Header_Straight_1x01_Pitch2.54mm, Pin_Headers:Pin_Header_Straight_1x01_Pitch2.54mm, F.Cu at (72.9, 131.4)
- added REF**: Pin_Header_Straight_1x01_Pitch2.54mm, Pin_Headers:Pin_Header_Straight_1x01_Pitch2.54mm, F.Cu at (92.7, 161.5)
- added REF**: Pin_Header_Straight_1x01_Pitch2.54mm, Pin_Headers:Pin_Header_Straight_1x01_Pitch2.54mm, F.Cu at (97.7, 162.5)
- added REF**: Pin_Header_Straight_1x01_Pitch2.54mm, Pin_Headers:Pin_Header_Straight_1x01_Pitch2.54mm, F.Cu at (102.6, 163.2)
- added REF**: Pin_Header_Straight_1x01_Pitch2.54mm, Pin_Headers:Pin_Header_Straight_1x01_Pitch2.54mm, F.Cu at (107.6, 163.6)
- added REF**: Pin_Header_Straight_1x01_Pitch2.54mm, Pin_Headers:Pin_Header_Straight_1x01_Pitch2.54mm, F.Cu at (112.7, 163.4)
- added REF**: Pin_Header_Straight_1x01_Pitch2.54mm, Pin_Headers:Pin_Header_Straight_1x01_Pitch2.54mm, F.Cu at (117.6, 163.2)
- added REF** (x2): Pin_Header_Straight_1x01_Pitch2.54mm, Pin_Headers:Pin_Header_Straight_1x01_Pitch2.54mm, F.Cu at (127.7, 161.2)
- added REF**: Pin_Header_Straight_1x01_Pitch2.54mm, Pin_Headers:Pin_Header_Straight_1x01_Pitch2.54mm, F.Cu at (122.7, 162.4)
- added REF**: Pin_Header_Straight_1x01_Pitch2.54mm, Pin_Headers:Pin_Header_Straight_1x01_Pitch2.54mm, F.Cu at (92.7, 131.4)
- added REF**: Pin_Header_Straight_1x01_Pitch2.54mm, Pin_Headers:Pin_Header_Straight_1x01_Pitch2.54mm, F.Cu at (148.6, 76.2)
- added REF**: Pin_Header_Straight_1x01_Pitch2.54mm, Pin_Headers:Pin_Header_Straight_1x01_Pitch2.54mm, F.Cu at (97.7, 131.4)
- added REF**: Pin_Header_Straight_1x01_Pitch2.54mm, Pin_Headers:Pin_Header_Straight_1x01_Pitch2.54mm, F.Cu at (102.6, 131.4)
- added REF**: Pin_Header_Straight_1x01_Pitch2.54mm, Pin_Headers:Pin_Header_Straight_1x01_Pitch2.54mm, F.Cu at (107.6, 131.4)
- added REF**: Pin_Header_Straight_1x01_Pitch2.54mm, Pin_Headers:Pin_Header_Straight_1x01_Pitch2.54mm, F.Cu at (112.6, 131.4)
- added REF**: Pin_Header_Straight_1x01_Pitch2.54mm, Pin_Headers:Pin_Header_Straight_1x01_Pitch2.54mm, F.Cu at (117.6, 131.4)
- added REF**: Pin_Header_Straight_1x01_Pitch2.54mm, Pin_Headers:Pin_Header_Straight_1x01_Pitch2.54mm, F.Cu at (122.7, 131.4)
- added REF**: Pin_Header_Straight_1x01_Pitch2.54mm, Pin_Headers:Pin_Header_Straight_1x01_Pitch2.54mm, F.Cu at (127.7, 131.4)
- added REF**: Pin_Header_Straight_1x01_Pitch2.54mm, Pin_Headers:Pin_Header_Straight_1x01_Pitch2.54mm, F.Cu at (72.9, 111.3)
- added REF**: Pin_Header_Straight_1x01_Pitch2.54mm, Pin_Headers:Pin_Header_Straight_1x01_Pitch2.54mm, F.Cu at (72.9, 106.3)
- added REF**: Pin_Header_Straight_1x01_Pitch2.54mm, Pin_Headers:Pin_Header_Straight_1x01_Pitch2.54mm, F.Cu at (73.0, 101.2)
- added REF**: Pin_Header_Straight_1x01_Pitch2.54mm, Pin_Headers:Pin_Header_Straight_1x01_Pitch2.54mm, F.Cu at (148.6, 81.2)
- added REF**: Pin_Header_Straight_1x01_Pitch2.54mm, Pin_Headers:Pin_Header_Straight_1x01_Pitch2.54mm, F.Cu at (72.9, 96.2)
- added REF**: Pin_Header_Straight_1x01_Pitch2.54mm, Pin_Headers:Pin_Header_Straight_1x01_Pitch2.54mm, F.Cu at (72.9, 91.2)
- added REF**: Pin_Header_Straight_1x01_Pitch2.54mm, Pin_Headers:Pin_Header_Straight_1x01_Pitch2.54mm, F.Cu at (72.9, 86.2)
- added REF**: Pin_Header_Straight_1x01_Pitch2.54mm, Pin_Headers:Pin_Header_Straight_1x01_Pitch2.54mm, F.Cu at (72.9, 81.3)
- added REF**: Pin_Header_Straight_1x01_Pitch2.54mm, Pin_Headers:Pin_Header_Straight_1x01_Pitch2.54mm, F.Cu at (72.9, 76.3)
- added REF** (x2): Pin_Header_Straight_1x01_Pitch2.54mm, Pin_Headers:Pin_Header_Straight_1x01_Pitch2.54mm, F.Cu at (43.2, 111.3)
- added REF**: Pin_Header_Straight_1x01_Pitch2.54mm, Pin_Headers:Pin_Header_Straight_1x01_Pitch2.54mm, F.Cu at (42.0, 106.3)
- added REF**: Pin_Header_Straight_1x01_Pitch2.54mm, Pin_Headers:Pin_Header_Straight_1x01_Pitch2.54mm, F.Cu at (41.2, 101.2)
- added REF**: Pin_Header_Straight_1x01_Pitch2.54mm, Pin_Headers:Pin_Header_Straight_1x01_Pitch2.54mm, F.Cu at (40.9, 96.3)
- added REF**: Pin_Header_Straight_1x01_Pitch2.54mm, Pin_Headers:Pin_Header_Straight_1x01_Pitch2.54mm, F.Cu at (148.5, 86.3)
- added REF**: Pin_Header_Straight_1x01_Pitch2.54mm, Pin_Headers:Pin_Header_Straight_1x01_Pitch2.54mm, F.Cu at (40.8, 91.2)
- added REF**: Pin_Header_Straight_1x01_Pitch2.54mm, Pin_Headers:Pin_Header_Straight_1x01_Pitch2.54mm, F.Cu at (41.2, 86.2)
- added REF**: Pin_Header_Straight_1x01_Pitch2.54mm, Pin_Headers:Pin_Header_Straight_1x01_Pitch2.54mm, F.Cu at (41.9, 81.3)
- added REF**: Pin_Header_Straight_1x01_Pitch2.54mm, Pin_Headers:Pin_Header_Straight_1x01_Pitch2.54mm, F.Cu at (42.9, 76.3)
- added REF**: Pin_Header_Straight_1x01_Pitch2.54mm, Pin_Headers:Pin_Header_Straight_1x01_Pitch2.54mm, F.Cu at (127.7, 25.7)
- added REF**: Pin_Header_Straight_1x01_Pitch2.54mm, Pin_Headers:Pin_Header_Straight_1x01_Pitch2.54mm, F.Cu at (122.7, 24.7)
- added REF**: Pin_Header_Straight_1x01_Pitch2.54mm, Pin_Headers:Pin_Header_Straight_1x01_Pitch2.54mm, F.Cu at (117.7, 24.0)
- added REF**: Pin_Header_Straight_1x01_Pitch2.54mm, Pin_Headers:Pin_Header_Straight_1x01_Pitch2.54mm, F.Cu at (112.7, 23.6)
- added REF**: Pin_Header_Straight_1x01_Pitch2.54mm, Pin_Headers:Pin_Header_Straight_1x01_Pitch2.54mm, F.Cu at (107.7, 23.8)
- added REF**: Pin_Header_Straight_1x01_Pitch2.54mm, Pin_Headers:Pin_Header_Straight_1x01_Pitch2.54mm, F.Cu at (102.7, 24.1)
- added REF**: Pin_Header_Straight_1x01_Pitch2.54mm, Pin_Headers:Pin_Header_Straight_1x01_Pitch2.54mm, F.Cu at (148.6, 91.3)
- added REF**: Pin_Header_Straight_1x01_Pitch2.54mm, Pin_Headers:Pin_Header_Straight_1x01_Pitch2.54mm, F.Cu at (92.6, 26.0)
- added REF**: Pin_Header_Straight_1x01_Pitch2.54mm, Pin_Headers:Pin_Header_Straight_1x01_Pitch2.54mm, F.Cu at (97.6, 24.8)
- added REF**: Pin_Header_Straight_1x01_Pitch2.54mm, Pin_Headers:Pin_Header_Straight_1x01_Pitch2.54mm, F.Cu at (92.7, 26.0)
- added REF**: Pin_Header_Straight_1x01_Pitch2.54mm, Pin_Headers:Pin_Header_Straight_1x01_Pitch2.54mm, F.Cu at (148.6, 96.3)
- added REF**: MountingHole_3.2mm_M3, Mounting_Holes:MountingHole_3.2mm_M3, F.Cu at (64.7, 47.8)
- added REF**: MountingHole_3.2mm_M3, Mounting_Holes:MountingHole_3.2mm_M3, F.Cu at (156.6, 47.9)
- added REF**: MountingHole_3.2mm_M3, Mounting_Holes:MountingHole_3.2mm_M3, F.Cu at (156.6, 139.8)
- added REF**: MountingHole_3.2mm_M3, Mounting_Holes:MountingHole_3.2mm_M3, F.Cu at (64.5, 139.8)
- added REF**: Pin_Header_Straight_1x01_Pitch2.54mm, Pin_Headers:Pin_Header_Straight_1x01_Pitch2.54mm, F.Cu at (148.6, 101.3)
- added REF**: Pin_Header_Straight_1x01_Pitch2.54mm, Pin_Headers:Pin_Header_Straight_1x01_Pitch2.54mm, F.Cu at (148.6, 106.2)
Routing:
- net (no net): track 0.00 -> 995.3 mm
Other:
- net class Default: trace_width 0.25 -> 0.6
