File: muon_geiger/geiger_mounts/geiger_mounts.kicad_pcb (KiCad board)
At the start: 2 copper layers, 32 x 133.1 mm, 22 parts

Commit message: finalising
Routing:
- net (no net): track 32.1 -> 117.0 mm
Changed lines of the file:
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@@
     (thickness 1.6)
     (drawings 22)
-    (tracks 11)
+    (tracks 20)
     (zones 0)
     (modules 22)
@@
     (visible_elements 7FFFFFFF)
     (pcbplotparams
-      (layerselection 0x00030_ffffffff)
+      (layerselection 0x010c0_ffffffff)
       (usegerberextensions false)
+      (usegerberattributes true)
+      (usegerberadvancedattributes true)
       (excludeedgelayer true)
       (linewidth 0.100000)
@@
       (outputformat 1)
       (mirror false)
-      (drillshape 1)
+      (drillshape 0)
       (scaleselection 1)
       (outputdirectory /root/projects/shift_register/core-crt-muon/muon_geiger/geiger_mounts/))
@@
   (gr_line (start 62.5 36.1) (end 62.5 169.1) (angle 90) (layer Edge.Cuts) (width 0.15))
   (gr_line (start 30.5 36.1) (end 62.5 36.1) (angle 90) (layer Edge.Cuts) (width 0.15))
+  (segment (start 36 144.55) (end 50.42 144.55) (width 0.6) (layer B.Cu) (net 0) (status C00000))
+  (segment (start 50.42 132.5) (end 36 132.5) (width 0.6) (layer B.Cu) (net 0) (status C00000))
+  (segment (start 42.8 120.5) (end 50.42 120.5) (width 0.6) (layer B.Cu) (net 0) (status C00000))
+  (segment (start 36 120.5) (end 42.8 120.5) (width 0.6) (layer B.Cu) (net 0) (status C00000))
+  (segment (start 36 108.35) (end 42.8 108.35) (width 0.6) (layer B.Cu) (net 0) (status C00000))
+  (segment (start 36 96.35) (end 50.42 96.35) (width 0.6) (layer B.Cu) (net 0) (status C00000))
+  (segment (start 36 84.2) (end 42.8 84.2) (width 0.6) (layer B.Cu) (net 0) (status C00000))
+  (segment (start 36 72.4) (end 42.8 72.4) (width 0.6) (layer B.Cu) (net 0) (status C00000))
+  (segment (start 36 60.6) (end 42.8 60.6) (width 0.6) (layer B.Cu) (net 0) (status C00000))
   (segment (start 50.37 144.45) (end 50.47 144.55) (width 0.6) (layer B.Cu) (net 0) (status C00000))
   (segment (start 50.32 132.45) (end 50.37 132.5) (width 0.6) (layer B.Cu) (net 0) (status C00000))
